File: HD1416.kicad_pcb (KiCad board)
At the start: 2 copper layers, 97.8 x 97.8 mm, 40 parts, among them J1 AudioJack2, Q1 MPSA20, Q2 MPSA20, Q3 BC547A

Commit message: Updates to PCBNew
Parts:
- removed R8: pot_lin, Connector_PinHeader_2.54mm:PinHeader_1x03_P2.54mm_Vertical
- H10, H11, H3, H4, H5, H6, H7, H8, H9: footprint Connector_Wire:SolderWire-2.5sqmm_1x01_D2.4mm_OD3.6mm -> Connector_Wire:SolderWire-0.5sqmm_1x01_D0.9mm_OD2.3mm
- J1: footprint Connector_Audio:Jack_6.35mm_Neutrik_NJ2FD-V_Vertical -> Connector_Wire:SolderWire-0.5sqmm_1x02_P4.8mm_D0.9mm_OD2.3mm
- R3: value pot_lin2 -> 500k
- moved H6 74.9 mm to (108.0, 88.3)
- moved H8 64.8 mm to (97.8, 88.3)
- moved H3 64.5 mm to (122.6, 88.3)
- moved H4 50.2 mm to (118.1, 88.3)
- moved H7 49.1 mm to (102.9, 88.3)
- moved H5 37.5 mm to (113.0, 88.3)
- moved J1 25.6 mm to (124.5, 96.5)
- moved H11 23.4 mm to (43.2, 160.0)
- moved H9 22.2 mm to (43.2, 145.4)
- moved R6 13.8 mm to (99.1, 94.0)
- moved C5 5.72 mm to (104.1, 106.6), turned to 90 degrees
- moved H10 5.08 mm to (43.2, 152.4)
- moved LS1 2.01 mm to (111.1, 95.9)
- moved TP2 1.91 mm to (43.2, 111.1)
- moved C4 1.78 mm to (85.1, 113.0)
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Connections:
- C1 pad 2: GND -> Net-(C1-Pad2)
- H10 pad 1: GND -> Net-(C1-Pad2)
- H9 pad 1: GND -> Net-(C1-Pad2)
Other:
- board text added: "S"
- board text added: "T"
