File: HD1416.kicad_pcb (KiCad board)
At the start: 2 copper layers, 97.8 x 97.8 mm, 32 parts, among them J2 ST, Q1 MPSA20, Q2 MPSA20, Q3 BC547A

Commit message: updates to schematic
Parts:
- added J2: "GND", Connector_Wire:SolderWire-0.5sqmm_1x01_D0.9mm_OD2.3mm, F.Cu at (44.4, 160.0)
- J1: renamed from J2; value ST -> "A"
- moved LS1 7.91 mm to (111.5, 104.4)
- moved R5 7.91 mm to (84.9, 94.2)
- moved R9 7.91 mm to (116.6, 109.4)
- moved C1 7.91 mm to (44.2, 145.0)
- moved C2 7.91 mm to (69.6, 116.8)
- moved C3 7.91 mm to (64.5, 112.0)
- moved C4 7.91 mm to (86.2, 120.9)
- moved C5 7.91 mm to (105.2, 114.5)
- moved J1 7.91 mm to (44.2, 153.3)
- moved Q3 7.91 mm to (113.4, 115.2)
- moved R1 7.91 mm to (51.2, 95.1)
- moved R4 7.91 mm to (66.5, 104.4)
- moved TP1 7.91 mm to (44.2, 112.0)
- moved TP2 7.91 mm to (44.2, 119.0)
- moved TP6 7.91 mm to (123.0, 117.1)
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- renumbered H8 to J3, H7 to J4, H6 to J5, H4 to J6, H5 to J7, H3 to J8
Routing:
- net GND: track 174.5 -> 0.00 mm
- net VCC: track 100.2 -> 0.00 mm
- net (no net): track 54.5 -> 0.00 mm
- net Net-(Q1-B): track 39.7 -> 0.00 mm
- net /astable2: track 35.8 -> 0.00 mm
- net Net-(Q3-B): track 35.6 -> 0.00 mm
- net Net-(Q2-B): track 30.1 -> 0.00 mm
- net Net-(J3-Pin_1): track 28.6 -> 0.00 mm
- net /astable1: track 27.5 -> 0.00 mm
- net /speaker: track 20.1 -> 0.00 mm
- net Net-(D1-A): track 12.7 -> 0.00 mm
- net Net-(R3-Pad2): track 7.88 -> 0.00 mm
- removed copper zone on B.Cu, net GND
- removed copper zone on F.Cu, net GND
Other:
- board text added: "{dblquote}G{dblquote}"
- board text added: "{dblquote}H{dblquote}"
