File: HD1416.kicad_sch (KiCad schematic)
At the start: 36 parts, among them J1 AudioJack2, Q1 MPSA20, Q2 MPSA20, Q3 BC547A

Commit message: routing board and improving 3D
Parts:
- C2: value .005u -> (none); footprint Capacitor_THT:C_Rect_L9.0mm_W2.5mm_P7.50mm_MKT -> (none)
- H10, H11, H3, H4, H5, H6, H7, H8, H9: footprint (none) -> Connector_Wire:SolderWire-0.5sqmm_1x01_D0.9mm_OD2.3mm
- J1: footprint (none) -> Connector_Wire:SolderWire-0.5sqmm_1x02_P4.8mm_D0.9mm_OD2.3mm
- LS1: footprint Buzzer_Beeper:Speaker_CUI_CMR-1206S-67 -> (none)
- R3: value (none) -> 500k; footprint (none) -> footprints:3299X-1-504LF
- R8: value (none) -> 25k
Connections:
- net +9 renamed VCC
- net node5: no longer names the net of C2.2, Q1.2 (B), R2.2, TP2.1
- net node6: no longer names the net of C3.2, Q2.2 (B), R4.2, TP3.1
Changed lines of the file:
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@@
     (effects (font (size 1.27 1.27)) (justify left bottom))
-  )
-  (label "node6" (at 154.94 96.52 0)
-    (effects (font (size 1.27 1.27) italic) (justify left bottom))
   )
   (label "speaker" (at 251.46 91.44 0)
     (effects (font (size 1.27 1.27)) (justify left bottom))
   )
-  (label "node5" (at 104.14 115.57 0)
-    (effects (font (size 1.27 1.27) italic) (justify left bottom))
-  )
   (label "astable2" (at 179.07 92.71 0)
     (effects (font (size 1.27 1.27) italic) (justify left bottom))
   )
-  (global_label "+9" (shape input) (at 86.36 81.28 180) (fields_autoplaced)
+  (global_label "VCC" (shape input) (at 86.36 81.28 180) (fields_autoplaced)
     (effects (font (size 1.27 1.27)) (justify right))
-    (property "Intersheet References" "${INTERSHEET_REFS}" (id 0) (at 81.165 81.2006 0)
+    (property "Intersheet References" "${INTERSHEET_REFS}" (id 0) (at 80.3183 81.2006 0)
       (effects (font (size 1.27 1.27)) (justify right) hide)
     )
   )
-  (global_label "+9" (shape input) (at 25.4 87.63 90) (fields_autoplaced)
+  (global_label "VCC" (shape input) (at 25.4 87.63 90) (fields_autoplaced)
     (effects (font (size 1.27 1.27)) (justify left))
-    (property "Intersheet References" "${INTERSHEET_REFS}" (id 0) (at 25.3206 82.435 90)
+    (property "Intersheet References" "${INTERSHEET_REFS}" (id 0) (at 25.3206 81.5883 90)
       (effects (font (size 1.27 1.27)) (justify left) hide)
     )
@@
     (in_bom yes) (on_board yes) (fields_autoplaced)
     (property "Reference" "R8" (id 0) (at 196.85 163.83 90))
-    (property "Value" "" (id 1) (at 196.85 166.37 90))
+    (property "Value" "25k" (id 1) (at 196.85 166.37 90))
     (property "Footprint" "" (id 2) (at 196.85 160.02 0)
       (effects (font (size 1.27 1.27)) hide)
@@
       (effects (font (size 1.27 1.27)) (justify left))
     )
-    (property "Footprint" "" (id 2) (at 67.31 110.49 0)
+    (property "Footprint" "Connector_Wire:SolderWire-0.5sqmm_1x01_D0.9mm_OD2.3mm" (id 2) (at 67.31 110.49 0)
       (effects (font (size 1.27 1.27)) hide)
     )
@@
     (in_bom yes) (on_board yes) (fields_autoplaced)
     (property "Reference" "C2" (id 0) (at 121.9136 109.22 90))
-    (property "Value" ".005u" (id 1) (at 121.9136 111.76 90))
-    (property "Footprint" "Capacitor_THT:C_Rect_L9.0mm_W2.5mm_P7.50mm_MKT" (id 2) (at 121.92 115.57 0)
+    (property "Value" "" (id 1) (at 121.9136 111.76 90))
+    (property "Footprint" "" (id 2) (at 121.92 115.57 0)
       (effects (font (size 1.27 1.27)) hide)
     )
@@
       (effects (font (size 1.27 1.27)) (justify left))
     )
-    (property "Footprint" "" (id 2) (at 59.69 110.49 0)
+    (property "Footprint" "Connector_Wire:SolderWire-0.5sqmm_1x01_D0.9mm_OD2.3mm" (id 2) (at 59.69 110.49 0)
       (effects (font (size 1.27 1.27)) hide)
     )
@@
     (property "Reference" "H5" (id 0) (at 215.9 143.51 90))
     (property "Value" "E" (id 1) (at 215.9 151.13 90))
-    (property "Footprint" "" (id 2) (at 217.17 147.32 0)
+    (property "Footprint" "Connector_Wire:SolderWire-0.5sqmm_1x01_D0.9mm_OD2.3mm" (id 2) (at 217.17 147.32 0)
       (effects (font (size 1.27 1.27)) hide)
     )
@@
     (property "Reference" "H8" (id 0) (at 189.23 143.51 90))
     (property "Value" "B" (id 1) (at 189.23 151.13 90))
-    (property "Footprint" "" (id 2) (at 190.5 147.32 0)
+    (property "Footprint" "Connector_Wire:SolderWire-0.5sqmm_1x01_D0.9mm_OD2.3mm" (id 2) (at 190.5 147.32 0)
       (effects (font (size 1.27 1.27)) hide)
     )
@@
       (effects (font (size 1.27 1.27)) (justify left))
     )
-    (property "Footprint" "" (id 2) (at 224.79 147.32 0)
+    (property "Footprint" "Connector_Wire:SolderWire-0.5sqmm_1x01_D0.9mm_OD2.3mm" (id 2) (at 224.79 147.32 0)
       (effects (font (size 1.27 1.27)) hide)
     )
@@
       (effects (font (size 1.27 1.27)) (justify left))
     )
-    (property "Footprint" "" (id 2) (at 203.2 147.32 0)
+    (property "Footprint" "Connector_Wire:SolderWire-0.5sqmm_1x01_D0.9mm_OD2.3mm" (id 2) (at 203.2 147.32 0)
       (effects (font (size 1.27 1.27)) hide)
     )
@@
       (effects (font (size 1.27 1.27)) (justify left))
     )
-    (property "Footprint" "Buzzer_Beeper:Speaker_CUI_CMR-1206S-67" (id 2) (at 256.54 86.36 0)
+    (property "Footprint" "" (id 2) (at 256.54 86.36 0)
       (effects (font (size 1.27 1.27)) hide)
     )
@@
       (effects (font (size 1.27 1.27)) (justify left))
     )
-    (property "Footprint" "" (id 2) (at 219.71 160.02 0)
+    (property "Footprint" "Connector_Wire:SolderWire-0.5sqmm_1x02_P4.8mm_D0.9mm_OD2.3mm" (id 2) (at 219.71 160.02 0)
       (effects (font (size 1.27 1.27)) hide)
     )
@@
       (effects (font (size 1.27 1.27)) (justify left))
     )
-    (property "Footprint" "" (id 2) (at 52.07 110.49 0)
+    (property "Footprint" "Connector_Wire:SolderWire-0.5sqmm_1x01_D0.9mm_OD2.3mm" (id 2) (at 52.07 110.49 0)
       (effects (font (size 1.27 1.27)) hide)
     )
@@
       (effects (font (size 1.27 1.27)) (justify right))
     )
-    (property "Value" "" (id 1) (at 137.16 88.8999 0)
-      (effects (font (size 1.27 1.27)) (justify right))
-    )
-    (property "Footprint" "" (id 2) (at 139.7 87.63 0)
+    (property "Value" "500k" (id 1) (at 137.16 88.8999 0)
+      (effects (font (size 1.27 1.27)) (justify right))
+    )
+    (property "Footprint" "footprints:3299X-1-504LF" (id 2) (at 139.7 87.63 0)
       (effects (font (size 1.27 1.27)) hide)
     )
@@
       (effects (font (size 1.27 1.27)) (justify right))
     )
-    (property "Footprint" "" (id 2) (at 210.82 130.81 0)
+    (property "Footprint" "Connector_Wire:SolderWire-0.5sqmm_1x01_D0.9mm_OD2.3mm" (id 2) (at 210.82 130.81 0)
       (effects (font (size 1.27 1.27)) hide)
     )
@@
       (effects (font (size 1.27 1.27)) (justify right))
     )
-    (property "Footprint" "" (id 2) (at 196.85 146.05 0)
+    (property "Footprint" "Connector_Wire:SolderWire-0.5sqmm_1x01_D0.9mm_OD2.3mm" (id 2) (at 196.85 146.05 0)
       (effects (font (size 1.27 1.27)) hide)
     )
@@
     )
     (path "/24d20a7d-c0ed-4f53-8c3d-0c655e1ebdd0"
-      (reference "C2") (unit 1) (value ".005u") (footprint "Capacitor_THT:C_Rect_L9.0mm_W2.5mm_P7.50mm_MKT")
+      (reference "C2") (unit 1) (value ".005u") (footprint "footprints:C315C103K5R5TA7303")
     )
     (path "/ba42d2d6-895c-44b2-8c3d-341bfc8b747d"
@@
     )
     (path "/7a8480ae-1026-4245-ab88-e1d30520ed35"
-      (reference "LS1") (unit 1) (value "50") (footprint "Buzzer_Beeper:Speaker_CUI_CMR-1206S-67")
+      (reference "LS1") (unit 1) (value "50") (footprint "Connector_Wire:SolderWire-0.5sqmm_1x02_P4.8mm_D0.9mm_OD2.3mm")
     )
     (path "/7d61c4fe-379c-49a7-a6d8-6a9306baf197"

Commit message: improved sch pcb 3d
Parts:
- added SW1, SW?: (no value), symbol Switch:SW_SPST
- C2: value (none) -> .005u; footprint (none) -> footprints:C315C103K5R5TA7303
- LS1: footprint (none) -> Connector_Wire:SolderWire-0.5sqmm_1x02_P4.8mm_D0.9mm_OD2.3mm
Connections:
- net GND: now also SW1.2 (B)
- net at C5.1, H4.1, H5.1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: now also H3.1, J1.S, R9.2
- net at C1.2, H10.1, H9.1: now also SW1.1 (A)
Other:
- moved on the sheet: C1, D1, H10, H11, H4, H5, H9, V1

Commit message: updated modeling
Parts:
- gave numbers to parts that had none: 1
Changed lines of the file:
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@@
   (symbol (lib_id "Switch:SW_SPST") (at 170.18 123.19 0) (unit 1)
     (in_bom yes) (on_board yes) (fields_autoplaced)
-    (property "Reference" "SW?" (id 0) (at 170.18 116.84 0))
+    (property "Reference" "SW2" (id 0) (at 170.18 116.84 0))
     (property "Value" "" (id 1) (at 170.18 119.38 0))
     (property "Footprint" "" (id 2) (at 170.18 123.19 0)
@@
     )
     (path "/5ecea6c7-cbcd-4340-9db8-55b54a886e1e"
-      (reference "SW?") (unit 1) (value "SW_SPST") (footprint "")
+      (reference "SW2") (unit 1) (value "SW_SPST") (footprint "")
     )
     (path "/4d4a752b-cc56-447b-9862-f2677b2033db"
