File: HD1416.kicad_sch (KiCad schematic)
At the start: 35 parts, among them J2 ST, J3 AudioJack3, Q1 MPSA20, Q2 MPSA20, Q3 BC547A, SW1 ${SIM.PARAMS}

Commit message: changes to folder organization
Parts:
- C3: value .01u -> .01
Changed lines of the file:
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@@
 			)
 		)
-		(property "Sim.Library" "Pot.lib"
+		(property "Sim.Library" "hd1416-spice-models\\Pot.lib"
 			(at 196.85 160.02 0)
 			(effects
@@
 		(property "Sim.Pins" "1=1 2=2 3=3"
 			(at 0 0 0)
+			(effects
+				(font
+					(size 1.27 1.27)
+				)
+				(hide yes)
+			)
+		)
+		(property "Sim.Device" "SUBCKT"
+			(at 196.85 160.02 0)
 			(effects
 				(font
@@
 			)
 		)
-		(property "Sim.Device" "SPICE"
+		(property "Sim.Device" "NPN"
 			(at 95.25 115.57 0)
 			(effects
@@
 			)
 		)
-		(property "Sim.Params" "type=\"Q\" model=\"MPSA20\" lib=\"standard.bjt\""
-			(at 0 0 0)
-			(effects
-				(font
-					(size 1.27 1.27)
-				)
-				(hide yes)
-			)
-		)
-		(property "Sim.Pins" "3=1 2=2 1=3"
+		(property "Sim.Pins" "1=E 2=B 3=C"
+			(at 95.25 115.57 0)
+			(effects
+				(font
+					(size 1.27 1.27)
+				)
+				(hide yes)
+			)
+		)
+		(property "Sim.Type" "VBIC"
 			(at 95.25 115.57 0)
 			(effects
@@
 			)
 		)
-		(property "Sim.Library" "Pot2.lib"
+		(property "Sim.Library" "hd1416-spice-models\\Pot2.lib"
 			(at 139.7 87.63 0)
 			(effects
@@
 		(property "Sim.Pins" "1=1 2=2 3=3"
 			(at 0 0 0)
+			(effects
+				(font
+					(size 1.27 1.27)
+				)
+				(hide yes)
+			)
+		)
+		(property "Sim.Device" "SUBCKT"
+			(at 139.7 87.63 0)
 			(effects
 				(font
@@
 			)
 		)
-		(property "Sim.Device" "SPICE"
+		(property "Sim.Device" "NPN"
 			(at 238.76 101.6 0)
 			(effects
@@
 			)
 		)
-		(property "Sim.Params" "type=\"Q\" model=\"BC547A\" lib=\"standard.bjt\""
-			(at 0 0 0)
-			(effects
-				(font
-					(size 1.27 1.27)
-				)
-				(hide yes)
-			)
-		)
-		(property "Sim.Pins" "3=1 2=2 1=3"
+		(property "Sim.Pins" "1=E 2=B 3=C"
+			(at 238.76 101.6 0)
+			(effects
+				(font
+					(size 1.27 1.27)
+				)
+				(hide yes)
+			)
+		)
+		(property "Sim.Type" "VBIC"
 			(at 238.76 101.6 0)
 			(effects
@@
 			)
 		)
-		(property "Value" ".01u"
+		(property "Value" ".01"
 			(at 146.0563 111.76 90)
 			(effects
@@
 			)
 		)
-		(property "Sim.Device" "SPICE"
+		(property "Sim.Device" "NPN"
 			(at 176.53 115.57 0)
 			(effects
@@
 			)
 		)
-		(property "Sim.Params" "type=\"Q\" model=\"MPSA20\" lib=\"standard.bjt\""
-			(at 0 0 0)
-			(effects
-				(font
-					(size 1.27 1.27)
-				)
-				(hide yes)
-			)
-		)
-		(property "Sim.Pins" "3=1 2=2 1=3"
+		(property "Sim.Pins" "1=E 2=B 3=C"
 			(at 176.53 115.57 0)
 			(effects
+				(font
+					(size 1.27 1.27)
+				)
+				(hide yes)
+			)
+		)
+		(property "Sim.Type" "VBIC"
+			(at 176.53 115.57 0)
+			(effects

Commit message: updates to schematic
Parts:
- added J2: "GND", Connector_Wire:SolderWire-0.5sqmm_1x01_D0.9mm_OD2.3mm, symbol Connector:Conn_01x01_Socket
- J1: renamed from J2; value ST -> "A"
- renumbered H8 to J3, H7 to J4, H6 to J5, H4 to J6, H5 to J7, H3 to J8, J3 to J9
Connections:
- net GND: now also J2.1 (Pin_1)
Other:
- note added: "+"
- note added: "-"
- note added: "A=top binding post"
- note added: "B=pot lug 3"
- note added: "C=phone pot lug 2"
- note added: "D=pot lug 1"
- note added: "E=phone jack lug 3"
- note added: "F=phone jack lug 2"
- note removed: "Spice model - J1 is 1 ohm R"
- moved on the sheet: SW1

Commit message: minor change
Connections:
- net GND: no longer D1.1 (K), V1.2
- new net: D1.1 (K), V1.2
Changed lines of the file:
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@@
 	)
 	(junction
-		(at 21.59 115.57)
-		(diameter 0)
-		(color 0 0 0 0)
-	)
-	(junction
 		(at 68.58 115.57)
 		(diameter 0)
@@
 	(wire
 		(pts
-			(xy 21.59 115.57) (xy 21.59 130.81)
-		)
-		(stroke
-			(width 0)
-			(type default)
-		)
-	)
-	(wire
-		(pts
 			(xy 38.1 115.57) (xy 38.1 120.65)
 		)
@@
 		(unit 1)
 		(exclude_from_sim yes)
-		(exclude_from_sim yes)
 		(in_bom yes)
 		(on_board no)
@@
 					(unit 1)
 				)
-			)
-		)
-	)
-	(symbol
-		(lib_id "power:GND")
-		(at 21.59 130.81 0)
-		(unit 1)
-		(exclude_from_sim no)
-		(in_bom yes)
-		(on_board yes)
-		(dnp no)
-		(fields_autoplaced yes)
-		(property "Reference" "#PWR01"
-			(at 21.59 137.16 0)
-			(effects
-				(font
-					(size 1.27 1.27)
-				)
-				(hide yes)
-			)
-		)
-		(property "Value" "GND"
-			(at 21.59 135.89 0)
-			(effects
-				(font
-					(size 1.27 1.27)
-				)
-			)
-		)
-		(property "Footprint" ""
-			(at 21.59 130.81 0)
-			(effects
-				(font
-					(size 1.27 1.27)
-				)
-				(hide yes)
-			)
-		)
-		(property "Datasheet" ""
-			(at 21.59 130.81 0)
-			(effects
-				(font
-					(size 1.27 1.27)
-				)
-				(hide yes)
-			)
-		)
-		(property "Description" "Power symbol creates a global label with name \"GND\" , ground"
-			(at 21.59 130.81 0)
-			(effects
-				(font
-					(size 1.27 1.27)
-				)
-				(hide yes)
-			)
-		)
-		(pin "1"
-		)
-		(instances
-			(project ""
-				(path "/e63e39d7-6ac0-4ffd-8aa3-1841a4541b55"
-					(reference "#PWR01")
-					(unit 1)
-				)
