File: HD1416_Oscillator_Board_sch.kicad_sch (KiCad schematic)
At the start: 37 parts, among them J1 AudioJack2, Q1 MPSA20, Q2 MPSA20, Q3 BC547A, SW1 SW_SPST

Commit message: catching up on all changes
Parts:
- removed C1, C3: .01u, Capacitor_THT:C_Disc_D3.8mm_W2.6mm_P2.50mm, symbol Device:C_Small
- removed C2: .005u, footprints:C315C103K5R5TA7303, symbol Device:C_Small
- removed C4: .1u, Capacitor_THT:C_Disc_D3.8mm_W2.6mm_P2.50mm, symbol Device:C_Small
- removed C5: .2u, Capacitor_THT:C_Disc_D3.8mm_W2.6mm_P2.50mm, symbol Device:C_Small
- removed D1: D1N4005, Diode_THT:D_DO-41_SOD81_P10.16mm_Horizontal, symbol Diode:1N4005
- removed H10: A, Connector_Wire:SolderWire-0.5sqmm_1x01_D0.9mm_OD2.3mm, symbol Mechanical:MountingHole_Pad
- removed H11: GND, Connector_Wire:SolderWire-0.5sqmm_1x01_D0.9mm_OD2.3mm, symbol Mechanical:MountingHole_Pad
- removed H3: 8200, Connector_Wire:SolderWire-0.5sqmm_1x01_D0.9mm_OD2.3mm, symbol Mechanical:MountingHole_Pad
- removed H4: F, Connector_Wire:SolderWire-0.5sqmm_1x01_D0.9mm_OD2.3mm, symbol Mechanical:MountingHole_Pad
- removed H5: E, Connector_Wire:SolderWire-0.5sqmm_1x01_D0.9mm_OD2.3mm, symbol Mechanical:MountingHole_Pad
- removed H6: D, Connector_Wire:SolderWire-0.5sqmm_1x01_D0.9mm_OD2.3mm, symbol Mechanical:MountingHole_Pad
- removed H7: C, Connector_Wire:SolderWire-0.5sqmm_1x01_D0.9mm_OD2.3mm, symbol Mechanical:MountingHole_Pad
- removed H8: B, Connector_Wire:SolderWire-0.5sqmm_1x01_D0.9mm_OD2.3mm, symbol Mechanical:MountingHole_Pad
- removed H9: ST, Connector_Wire:SolderWire-0.5sqmm_1x01_D0.9mm_OD2.3mm, symbol Mechanical:MountingHole_Pad
- removed J1: AudioJack2, Connector_Wire:SolderWire-0.5sqmm_1x02_P4.8mm_D0.9mm_OD2.3mm, symbol Connector:AudioJack2
- removed LS1: 50, Connector_Wire:SolderWire-0.5sqmm_1x02_P4.8mm_D0.9mm_OD2.3mm, symbol Device:Speaker
- removed Q1, Q2: MPSA20, Package_TO_SOT_THT:TO-92, symbol Transistor_BJT:2N2219
- removed Q3: BC547A, Package_TO_SOT_THT:TO-92, symbol Transistor_BJT:2N2219
- removed R1: (no value), symbol Device:R_Small_US
- removed R2: 220k, footprints:SFR16S0002203FR500, symbol Device:R_Small_US
- removed R3: 500k, footprints:3299X-1-504LF, symbol Device:R_Potentiometer_Trim_US
- removed R4: 68k, footprints:CFR-50JB-52-68K, symbol Device:R_Small_US
- removed R5: 5.6k, footprints:CFR-50JB-52-5K6, symbol Device:R_Small_US
- removed R6: 2.2k, footprints:CFM12JT2K20, symbol Device:R_Small_US
- removed R7: 33k, footprints:CFM12JT33K0, symbol Device:R_Small_US
- removed R8: 25k, symbol Device:R_Potentiometer_Trim_US
- removed R9: 8200, footprints:CF12JT8K20, symbol Device:R_Small_US
- removed SW1: SW_SPST, symbol Switch:SW_SPST
- removed TP1: 2.4, TestPoint:TestPoint_Pad_D2.0mm, symbol Connector:TestPoint_Flag
- removed TP2: -0.3, TestPoint:TestPoint_Pad_D2.0mm, symbol Connector:TestPoint_Flag
- removed TP3: -2.1, TestPoint:TestPoint_Pad_D2.0mm, symbol Connector:TestPoint_Flag
- removed TP4: 5.1, TestPoint:TestPoint_Pad_D2.0mm, symbol Connector:TestPoint_Flag
- removed TP5: 0.5, TestPoint:TestPoint_Pad_D2.0mm, symbol Connector:TestPoint_Flag
- removed TP6: 7.5, TestPoint:TestPoint_Pad_D2.0mm, symbol Connector:TestPoint_Flag
- removed V1: 9, footprints:BatteryHolder_MPD_BA9VPC_1xPP3 dem, symbol pspice:VSOURCE
- added C?: .005u, footprints:C315C103K5R5TA7303, symbol Device:C_Small
- added C?: .2u, Capacitor_THT:C_Disc_D3.8mm_W2.6mm_P2.50mm, symbol Device:C_Small
- added C?: .1u, Capacitor_THT:C_Disc_D3.8mm_W2.6mm_P2.50mm, symbol Device:C_Small
- added C? (x2): .01u, Capacitor_THT:C_Disc_D3.8mm_W2.6mm_P2.50mm, symbol Device:C_Small
- added D?: D1N4005, Diode_THT:D_DO-41_SOD81_P10.16mm_Horizontal, symbol Diode:1N4005
- added H?: GND, Connector_Wire:SolderWire-0.5sqmm_1x01_D0.9mm_OD2.3mm, symbol Mechanical:MountingHole_Pad
- added H?: ST, Connector_Wire:SolderWire-0.5sqmm_1x01_D0.9mm_OD2.3mm, symbol Mechanical:MountingHole_Pad
- added H?: B, Connector_Wire:SolderWire-0.5sqmm_1x01_D0.9mm_OD2.3mm, symbol Mechanical:MountingHole_Pad
- added H?: F, Connector_Wire:SolderWire-0.5sqmm_1x01_D0.9mm_OD2.3mm, symbol Mechanical:MountingHole_Pad
- added H?: D, Connector_Wire:SolderWire-0.5sqmm_1x01_D0.9mm_OD2.3mm, symbol Mechanical:MountingHole_Pad
- added H?: C, Connector_Wire:SolderWire-0.5sqmm_1x01_D0.9mm_OD2.3mm, symbol Mechanical:MountingHole_Pad
- added H?: A, Connector_Wire:SolderWire-0.5sqmm_1x01_D0.9mm_OD2.3mm, symbol Mechanical:MountingHole_Pad
- added H?: 8200, Connector_Wire:SolderWire-0.5sqmm_1x01_D0.9mm_OD2.3mm, symbol Mechanical:MountingHole_Pad
- added H?: E, Connector_Wire:SolderWire-0.5sqmm_1x01_D0.9mm_OD2.3mm, symbol Mechanical:MountingHole_Pad
- added J?: AudioJack2, Connector_Wire:SolderWire-0.5sqmm_1x02_P4.8mm_D0.9mm_OD2.3mm, symbol Connector:AudioJack2
- added LS?: 50, Connector_Wire:SolderWire-0.5sqmm_1x02_P4.8mm_D0.9mm_OD2.3mm, symbol Device:Speaker
- added Q? (x2): MPSA20, Package_TO_SOT_THT:TO-92, symbol Transistor_BJT:2N2219
- added Q?: BC547A, Package_TO_SOT_THT:TO-92, symbol Transistor_BJT:2N2219
- added R?: 25k, symbol Device:R_Potentiometer_Trim_US
- added R?: 220k, footprints:SFR16S0002203FR500, symbol Device:R_Small_US
- added R?: 5.6k, footprints:CFR-50JB-52-5K6, symbol Device:R_Small_US
- added R?: 2.2k, footprints:CFM12JT2K20, symbol Device:R_Small_US
- added R?: 68k, footprints:CFR-50JB-52-68K, symbol Device:R_Small_US
- added R?: 8200, footprints:CF12JT8K20, symbol Device:R_Small_US
- added R?: 33k, footprints:CFM12JT33K0, symbol Device:R_Small_US
- added R?: 10k, footprints:CFM12JT10K0, symbol Device:R_Small_US
- added R?: 500k, footprints:3299X-1-504LF, symbol Device:R_Potentiometer_Trim_US
- added SW?: SW_SPST, symbol Switch:SW_SPST
- added TP?: 7.5, TestPoint:TestPoint_Pad_D2.0mm, symbol Connector:TestPoint_Flag
- added TP?: 2.4, TestPoint:TestPoint_Pad_D2.0mm, symbol Connector:TestPoint_Flag
- added TP?: -0.3, TestPoint:TestPoint_Pad_D2.0mm, symbol Connector:TestPoint_Flag
- added TP?: 5.1, TestPoint:TestPoint_Pad_D2.0mm, symbol Connector:TestPoint_Flag
- added TP?: -2.1, TestPoint:TestPoint_Pad_D2.0mm, symbol Connector:TestPoint_Flag
- added TP?: 0.5, TestPoint:TestPoint_Pad_D2.0mm, symbol Connector:TestPoint_Flag
- added V?: 9, footprints:BatteryHolder_MPD_BA9VPC_1xPP3 dem, symbol pspice:VSOURCE
Connections:
- net GND: now also D?.1 (K), H?.1, H?.1, Q?.1 (E), Q?.1 (E), Q?.1 (E), R?.1, R?.2, R?.3, R?.3, SW?.2 (B), V?.2 (E2)
- net VCC: now also LS?.1, R?.1, R?.1, R?.1, R?.1, R?.1, V?.1 (E1)
- net astable1: now also C?.1, Q?.3 (C), R?.2, TP?.1
- net astable2: now also C?.1, C?.1, Q?.3 (C), R?.2, TP?.1
- net speaker: now also LS?.2, Q?.3 (C), TP?.1
- new net: C?.2, H?.1, R?.1
- new net: C?.1, H?.1, H?.1, H?.1, H?.1, J?.S, J?.T, R?.2, R?.2
- new net: C?.2, Q?.2 (B), R?.2, TP?.1 (x2)
- new net: C?.2, H?.1, H?.1, SW?.1 (A)
- new net: C?.2, Q?.2 (B), R?.1, R?.2, TP?.1
- new net: C?.1, D?.2 (A)
- new net: R?.1, R?.2
Other:
- title: HD1416 Code Oscillator -> (none)
